File: stm32g431cxux/stm32g431cxux.kicad_pcb (KiCad board)
At the start: 2 copper layers, 17.8 x 31.2 mm, 23 parts, among them J1 USB2.0_C_v3, J2 ProMicro-LeftPin-NoGND, J3 ProMicro-RightPin, SW1 SW_Push, U1 AMS1117-3.3, U2 STM32G431CBUx, Y1 24M

Commit message: before free routing
Routing:
- net +3V3: track 44.2 -> 55.1 mm
Changed lines of the file:
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@@
   (segment (start 71.882 39.624) (end 71.374 39.116) (width 0.25) (layer "B.Cu") (net 1))
   (segment (start 66.04 39.116) (end 71.374 39.116) (width 0.25) (layer "B.Cu") (net 1))
+  (segment (start 70.375 53.425) (end 70.4 53.45) (width 0.25) (layer "F.Cu") (net 3))
+  (segment (start 69.4775 53.925) (end 69.925 53.925) (width 0.25) (layer "F.Cu") (net 3))
+  (segment (start 70.4 53.45) (end 70.4 52.493) (width 0.25) (layer "F.Cu") (net 3))
   (segment (start 63.246 58.1565) (end 63.29 58.1125) (width 0.25) (layer "F.Cu") (net 3))
   (segment (start 69.5035 52.451) (end 69.4775 52.425) (width 0.25) (layer "F.Cu") (net 3))
   (segment (start 68.0955 45.0615) (end 68.0955 45.085) (width 0.25) (layer "F.Cu") (net 3))
+  (segment (start 70.4 52.493) (end 70.358 52.451) (width 0.25) (layer "F.Cu") (net 3))
   (segment (start 70.358 52.451) (end 69.5035 52.451) (width 0.25) (layer "F.Cu") (net 3))
+  (segment (start 69.925 53.925) (end 70.4 53.45) (width 0.25) (layer "F.Cu") (net 3))
   (segment (start 69.215 43.942) (end 68.0955 45.0615) (width 0.25) (layer "F.Cu") (net 3))
   (segment (start 63.246 58.928) (end 63.246 58.1565) (width 0.25) (layer "F.Cu") (net 3))
   (segment (start 62.6025 57.425) (end 61.743 57.425) (width 0.25) (layer "F.Cu") (net 3))
+  (segment (start 69.4775 53.425) (end 70.375 53.425) (width 0.25) (layer "F.Cu") (net 3))
   (segment (start 61.743 57.425) (end 61.722 57.404) (width 0.25) (layer "F.Cu") (net 3))
   (via (at 70.358 52.451) (size 0.6) (drill 0.35) (layers "F.Cu" "B.Cu") (net 3))
@@
   (segment (start 63.3735 58.8005) (end 63.246 58.928) (width 0.25) (layer "B.Cu") (net 3))
   (segment (start 68.58 44.577) (end 69.215 43.942) (width 0.25) (layer "B.Cu") (net 3))
+  (segment (start 70.612 47.244) (end 70.104 47.752) (width 0.25) (layer "B.Cu") (net 3))
   (segment (start 68.58 45.593) (end 68.58 48.895) (width 0.25) (layer "B.Cu") (net 3))
+  (segment (start 73.66 45.72) (end 72.644 45.72) (width 0.25) (layer "B.Cu") (net 3))
   (segment (start 68.58 45.593) (end 68.58 44.577) (width 0.25) (layer "B.Cu") (net 3))
   (segment (start 65.225 49.276) (end 65.225 50.874) (width 0.25) (layer "B.Cu") (net 3))
@@
   (segment (start 65.225 50.874) (end 65.786 51.435) (width 0.25) (layer "B.Cu") (net 3))
   (segment (start 63.5 57.404) (end 64.008 56.896) (width 0.25) (layer "B.Cu") (net 3))
+  (segment (start 68.58 45.593) (end 68.58 47.244) (width 0.25) (layer "B.Cu") (net 3))
   (segment (start 69.2155 52.451) (end 70.358 52.451) (width 0.25) (layer "B.Cu") (net 3))
   (segment (start 65.225 55.679) (end 64.8335 56.0705) (width 0.25) (layer "B.Cu") (net 3))
+  (segment (start 71.12 47.244) (end 70.612 47.244) (width 0.25) (layer "B.Cu") (net 3))
   (segment (start 65.225 50.874) (end 65.225 55.679) (width 0.25) (layer "B.Cu") (net 3))
   (segment (start 65.225 46.048) (end 64.77 45.593) (width 0.25) (layer "B.Cu") (net 3))
@@
   (segment (start 68.1995 51.435) (end 69.2155 52.451) (width 0.25) (layer "B.Cu") (net 3))
   (segment (start 68.58 45.593) (end 68.58 48.133) (width 0.25) (layer "B.Cu") (net 3))
+  (segment (start 68.58 47.244) (end 69.088 47.752) (width 0.25) (layer "B.Cu") (net 3))
   (segment (start 63.754 50.747) (end 65.225 49.276) (width 0.25) (layer "B.Cu") (net 3))
+  (segment (start 72.644 45.72) (end 71.12 47.244) (width 0.25) (layer "B.Cu") (net 3))
   (segment (start 65.225 49.276) (end 65.225 46.048) (width 0.25) (layer "B.Cu") (net 3))
   (segment (start 64.897 56.134) (end 64.897 58.0385) (width 0.25) (layer "B.Cu") (net 3))
@@
   (segment (start 61.722 57.404) (end 63.5 57.404) (width 0.25) (layer "B.Cu") (net 3))
   (segment (start 64.897 58.0385) (end 64.135 58.8005) (width 0.25) (layer "B.Cu") (net 3))
+  (segment (start 69.088 47.752) (end 70.104 47.752) (width 0.25) (layer "B.Cu") (net 3))
   (segment (start 64.8335 56.0705) (end 64.897 56.134) (width 0.25) (layer "B.Cu") (net 3))
   (segment (start 68.45 42.415) (end 68.45 42.676) (width 0.25) (layer "F.Cu") (net 7))

Commit message: before free routing
Routing:
- net Net-(U2-PF1): track 0.00 -> 6.55 mm, vias 0 -> 1
- net Net-(U2-PF0): track 0.00 -> 2.85 mm, vias 0 -> 1
Changed lines of the file:
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@@
   (segment (start 73.66 43.795) (end 73.66 43.18) (width 0.15) (layer "F.Cu") (net 30))
   (segment (start 66.255 46.55) (end 70.905 46.55) (width 0.15) (layer "F.Cu") (net 30))
+  (segment (start 65.29 59) (end 65.29 58.1125) (width 0.15) (layer "F.Cu") (net 35))
+  (via (at 65.29 59) (size 0.6) (drill 0.35) (layers "F.Cu" "B.Cu") (net 35))
+  (segment (start 65.722 59) (end 66.802 60.08) (width 0.15) (layer "B.Cu") (net 35))
+  (segment (start 65.29 59) (end 65.722 59) (width 0.15) (layer "B.Cu") (net 35))
+  (segment (start 65.79 58.74) (end 66.35 59.3) (width 0.15) (layer "F.Cu") (net 36))
+  (segment (start 65.79 58.1125) (end 65.79 58.74) (width 0.15) (layer "F.Cu") (net 36))
+  (segment (start 66.35 60.6) (end 66.95 61.2) (width 0.15) (layer "F.Cu") (net 36))
+  (segment (start 66.95 61.2) (end 68.2 61.2) (width 0.15) (layer "F.Cu") (net 36))
+  (segment (start 66.35 59.3) (end 66.35 60.6) (width 0.15) (layer "F.Cu") (net 36))
+  (via (at 68.2 61.2) (size 0.6) (drill 0.35) (layers "F.Cu" "B.Cu") (net 36))
+  (segment (start 68.472 61.2) (end 69.502 62.23) (width 0.15) (layer "B.Cu") (net 36))
+  (segment (start 68.2 61.2) (end 68.472 61.2) (width 0.15) (layer "B.Cu") (net 36))
   (zone (net 2) (net_name "GND") (layers "F&B.Cu") (hatch edge 0.5)
     (connect_pads (clearance 0.5))

Commit message: before free routing
Parts:
- moved C7 7.56 mm to (71.4, 60.9), turned to -90 degrees
- moved C8 7.51 mm to (64.0, 62.2), turned to 180 degrees
Routing:
- net +3V3: track 55.1 -> 59.6 mm, vias 4 -> 5
- net Net-(C8-Pad1): track 0.00 -> 2.05 mm
- net Net-(C7-Pad1): track 0.00 -> 1.92 mm

Commit message: before free routing
Parts:
- moved C2 5.39 mm to (64.2, 43.9)
- moved C3 4.61 mm to (60.4, 58.2), turned to -90 degrees
- moved C4 4.03 mm to (60.4, 50.2), turned to 90 degrees
- moved C6 0.74 mm to (63.9, 60.2), turned to 0 degrees
Routing:
- net +3V3: track 59.6 -> 85.6 mm
- net /D-: track 10.9 -> 5.68 mm

Commit message: before free routing
Parts:
- moved C2 8.24 mm to (71.9, 46.7), turned to -90 degrees
- moved C5 3.48 mm to (71.8, 53.2), turned to -90 degrees
Routing:
- net +3V3: track 85.6 -> 160.0 mm
- net /D-: track 5.68 -> 10.9 mm
Other:
- board size 17.8 x 31.2 mm -> 17.8 x 31.8 mm

Commit message: before free routing
Parts:
- C3, C4, C6: moved to F.Cu
- moved C6 1.52 mm to (62.4, 60.8), turned to 180 degrees
- moved Y1 0.07 mm to (68.2, 61.2)
Routing:
- net +3V3: track 160.0 -> 170.0 mm, vias 5 -> 6
- net Net-(U2-PF0): track 2.85 -> 1.01 mm
- net Net-(U2-PF1): track 6.55 -> 7.66 mm
- net +5V: track 56.0 -> 56.9 mm

Commit message: before free routing
Parts:
- moved R4 7.24 mm to (60.1, 55.0), turned to 90 degrees
- moved D1 1.09 mm to (62.6, 44.5)
- moved R3 1.09 mm to (62.6, 44.5)
- moved C4 0.45 mm to (60.1, 49.8)
- moved C3 0.25 mm to (60.1, 58.2)
- moved C5 0.15 mm to (72.0, 53.2)
Routing:
- net GND: track 0.00 -> 42.0 mm, vias 0 -> 2
- net +3V3: track 170.0 -> 161.0 mm
- net Net-(U2-PB8): track 0.00 -> 2.74 mm
- net Net-(D1-A): track 0.00 -> 1.85 mm, vias 0 -> 1
- net Net-(U2-PF0): track 1.01 -> 0.00 mm, vias 1 -> 0

Commit message: before free routing
Routing:
- net GND: vias 2 -> 4
Changed lines of the file:
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@@
   (segment (start 59.25 49.15) (end 59.775 49.15) (width 0.3) (layer "F.Cu") (net 2))
   (segment (start 59.775 49.15) (end 60.1 48.825) (width 0.3) (layer "F.Cu") (net 2))
+  (via (at 67.31 53.34) (size 0.6) (drill 0.35) (layers "F.Cu" "B.Cu") (net 2))
+  (via (at 64.77 53.34) (size 0.6) (drill 0.35) (layers "F.Cu" "B.Cu") (net 2))
   (via (at 60 66.35) (size 0.6) (drill 0.35) (layers "F.Cu" "B.Cu") (net 2))
   (via (at 59.25 49.15) (size 0.6) (drill 0.35) (layers "F.Cu" "B.Cu") (net 2))
